File: esp32-c3-mini.kicad_pcb (KiCad board)
At the start: 4 copper layers, 25 x 27.8 mm, 43 parts, among them J1 Conn_01x07_Pin, J2 Conn_01x07_Pin, P2 USB_C_Plug, SW1 SW_Push, SW2 SW_Push, U1 ME6211C33M5, U2 ESP32-C3, Y1 Crystal_GND24_Small

Commit message: Replace USB plug with USB-C receptacle
Replace the previous USB plug footprint with a USB_C_Receptacle_HRO_TYPE-C-31-M-12 footprint (USB2.0/PD). Update pad geometry, positions, orientations, silkscreen and UUIDs; remap nets/pin names from the old P2 plugin (P2-CC, P2-D+, P2-D-, P2-VCONN, etc.) to J3 equivalents and adjust pad sizes/types (SMD and thru-holes) accordingly. Remove generated Gerber outputs and add a production backup ZIP; update production artifacts (bom.csv, designators.csv, esp32-c3-mini.zip, netlist.ipc, positions.csv) to reflect the PCB changes.
Parts:
- removed P2: USB_C_Plug, Connector_USB:USB_C_Plug_Molex_105444
- added J3: USB_C_Receptacle_USB2.0_16P, Connector_USB:USB_C_Receptacle_HRO_TYPE-C-31-M-12, F.Cu at (124.4, 59.9)
- moved R10 2.01 mm to (124.3, 65.1)
- moved R9 2.00 mm to (126.3, 65.1)
- turned R12 to -90 degrees
Routing:
- net Net-(J3-D+-PadA6): track 4.14 -> 11.3 mm, vias 0 -> 2
- net Net-(J3-D--PadA7): track 4.62 -> 11.7 mm
- net Net-(J3-CC1): track 3.50 -> 8.76 mm
- net Net-(J3-CC2): track 4.11 -> 8.90 mm, vias 1 -> 0
- net GND: track 29.7 -> 27.4 mm
- net USB_D-: track 17.4 -> 15.4 mm
- net +5V: track 31.0 -> 30.7 mm, vias 0 -> 2
Other:
- board size 25 x 27.8 mm -> 25 x 33.2 mm

Commit message: Rotate USB-C footprint and update routing
Rotate the USB-C receptacle footprint 180° (update (at) coordinates and properties), mirror/update silkscreen/courtyard/fab lines and refresh fp UUIDs. Add/adjust board routing: new traces, vias and segments for CC1/CC2 and USB D+/D- nets, and reorganize GND and +5V segments (replace/relocate several vias and segments). Regenerate production artifacts: updated production zip, netlist and positions CSV, and add a production backup archive.
Parts:
- moved J3 1.69 mm to (124.4, 58.2), turned to 180 degrees
Routing:
- net +5V: track 30.7 -> 23.5 mm, vias 2 -> 0
- net Net-(J3-D--PadA7): track 11.7 -> 4.98 mm, vias 0 -> 2
- net Net-(J3-D+-PadA6): track 11.3 -> 4.61 mm
- net Net-(J3-CC1): track 8.76 -> 5.28 mm, vias 0 -> 2
- net Net-(J3-CC2): track 8.90 -> 6.60 mm, vias 0 -> 2
- net GND: vias 12 -> 11
Other:
- board size 25 x 33.2 mm -> 25 x 33.8 mm
